File: examples/prssine/eagle/prssine.sch (EAGLE design)
At the start: 8 parts

Commit message: Refactor to begin with common library, bugfix in ngspice.ulp to correctly compile prssine.sch
Other:
- note added: ".include yosys/prim_cells_ngspice.mod"
- note removed: ".include ../../../yosys/prim_cells_ngspice.mod"
Changed lines of the file:
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@@
 <sheet>
 <plain>
-<text x="81.28" y="-15.24" size="1.778" layer="100">.include ../../../yosys/prim_cells_ngspice.mod</text>
+<text x="81.28" y="-15.24" size="1.778" layer="100">.include yosys/prim_cells_ngspice.mod</text>
 <text x="81.28" y="-20.32" size="1.778" layer="110">.tran 50ns 50ms uic</text>
 </plain>
